File: PowerSupply.kicad_sch (KiCad schematic)
At the start: 56 parts

Commit message: optimization
Parts:
- added C19: 47uF, symbol Device:C_Polarized_Small
- added L1: 22uH, symbol Device:L_Small
- C1: renamed from C?; value 0,22uF -> 0,22uF 220V
- U1: renamed from U?; value L7815 -> L7818
- U2: renamed from U?; value L7915 -> L7918
- gave numbers to parts that had none: 53
Connections:
- net GND: now also C19.2
- net V-Raw: now also D6.2 (A), Q2.3 (E); no longer D6.1 (K), Q2.2 (C)
- net +Ub renamed VDD
- net -Ub renamed VSS
- net VSS: now also D6.1 (K), Q2.2 (C); no longer D6.2 (A), Q2.3 (E)
- net 5V: no longer names the net of C18.1, PS1.4 (+Vo)
- net 5V: now also L1.1; no longer C20.1
- net R_PWR+ renamed +5V
- net +5V: now also C20.1, C19.1, L1.2
- net R_PWR- renamed R_PWR
Other:
- moved on the sheet: C18, C20, PS1, Q2
