File: Whammy Amp Balanced.kicad_sch (KiCad schematic)
At the start: 7 parts

Commit message: optimization
Parts:
- added J?: Bal_Out, symbol Connector:AudioJack5
- added J?: AddIn_Conn, symbol Connector_Generic:Conn_02x12_Odd_Even
- added J?: Unbal_Out, symbol Connector:AudioJack3
- added K? (x3): G6S-2, symbol Relay:G6S-2
- TP?: footprint (none) -> TestPoint:TestPoint_Pad_D1.5mm
Connections:
- new net +5V: K?.1, K?.1, K?.1
- new net GND: J?.S, J?.S
- new net L+: J?.T, K?.8, K?.9
- new net L-: J?.R1, K?.5
- new net L_unbal+: J?.T, K?.8
- new net Out_L+: K?.9
- new net Out_L-: K?.4
- new net Out_R+: K?.9
- new net Out_R-: K?.4
- new net R+: J?.R2, K?.4, K?.8
- new net R-: J?.R3, K?.5
- new net R_Mute_L: K?.12
- new net R_Mute_R: K?.12
- new net R_Unbal: K?.12
- new net R_unbal+: J?.R, K?.3
- no-connect marks 0 -> 4
Other:
- removed sheet Amp
- added sheet amplifier_L (amplifier.kicad_sch)
- added sheet amplifier_R (amplifier.kicad_sch)
- sheet Power Supply ports: added 5V, R_PWR, V+, V-; removed none
- note added: "VDD - (+20V) VSS - (-20V) +5V"
- company: (none) -> ncAudio
- title: (none) -> NCBalWHAMMY
- moved on the sheet: C?, D?, R?, SW?, TP?
